File: SWR Protector.kicad_sch (KiCad schematic)
At the start: 27 parts, among them J1 Barrel_Jack, J2 Barrel_Jack, J3 transceiver, J4 antenna, K2 ATX209, Q1 2N3904, T1 1:12, T2 12:1 ???, U1 LM78L05_TO92, U2 LM358

Commit message: placed parts on PCB and wired them up.  DRC reports zero errors and a handful of warnings about overlapping silk screen.
Parts:
- RV1: footprint Resistor_THT:R_Axial_DIN0207_L6.3mm_D2.5mm_P7.62mm_Horizontal -> Potentiometer_THT:Potentiometer_Alpha_RD901F-40-00D_Single_Vertical
- T1, T2: footprint Transformer_THT:Transformer_Toroid_Horizontal_D18.0mm -> Transformer_THT:Transformer_Toroid_Horizontal_D9.0mm_Amidon-T30
Changed lines of the file:
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@@
   (title_block
     (title "SWR Protector WA7GIL")
-    (date "2023-05-06")
+    (date "2023-05-08")
     (rev "0.5")
   )
@@
       (effects (font (size 1.27 1.27) (color 255 0 0 1)) (justify left))
     )
-    (property "Footprint" "Transformer_THT:Transformer_Toroid_Horizontal_D18.0mm" (at 99.06 71.12 0)
+    (property "Footprint" "Transformer_THT:Transformer_Toroid_Horizontal_D9.0mm_Amidon-T30" (at 99.06 71.12 0)
       (effects (font (size 1.27 1.27)) hide)
     )
@@
       (effects (font (size 1.27 1.27)) (justify right))
     )
-    (property "Footprint" "Resistor_THT:R_Axial_DIN0207_L6.3mm_D2.5mm_P7.62mm_Horizontal" (at 121.92 146.05 0)
+    (property "Footprint" "Potentiometer_THT:Potentiometer_Alpha_RD901F-40-00D_Single_Vertical" (at 121.92 146.05 0)
       (effects (font (size 1.27 1.27)) hide)
     )
@@
       (effects (font (size 1.27 1.27)) (justify left))
     )
-    (property "Footprint" "Transformer_THT:Transformer_Toroid_Horizontal_D18.0mm" (at 73.66 45.72 0)
-      (effects (font (size 1.27 1.27)) hide)
-    )
+    (property "Footprint" "Transformer_THT:Transformer_Toroid_Horizontal_D9.0mm_Amidon-T30" (at 73.66 45.72 0)
+      (effects (font (size 1.27 1.27)) hide)
+    )

Commit message: Wider traces done.  FT37-43 oriented vertically with new footprint.
Parts:
- T1: footprint Transformer_THT:Transformer_Toroid_Horizontal_D9.0mm_Amidon-T30 -> FT37-43:FT37-43-TRANSFORMER
- T2: value 12:1 ??? -> 1:12; footprint Transformer_THT:Transformer_Toroid_Horizontal_D9.0mm_Amidon-T30 -> FT37-43:FT37-43-TRANSFORMER
Connections:
- net GND: now also T1.1 (AA), T2.2 (AB); no longer T1.4 (SB), T2.3 (SA)
- net at D3.2 (A), R5.2: now also T1.2 (AB), T2.4 (SB); no longer T1.3 (SA), T2.2 (AB)
- net at D4.2 (A), R6.1: now also T2.3 (SA); no longer T2.1 (AA)
- net at J3.1 (In): now also T1.4 (SB); no longer T1.2 (AB)
- new net: J4.1 (In), T1.3 (SA), T2.1 (AA)
Other:
- moved on the sheet: T1, T2
Changed lines of the file:
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@@
   (title_block
     (title "SWR Protector WA7GIL")
-    (date "2023-05-08")
-    (rev "0.5")
+    (date "2023-05-09")
+    (rev "0.6")
   )
   (junction (at 111.76 35.56) (diameter 0) (color 0 0 0 0)
@@
   )
   (junction (at 226.06 125.73) (diameter 0) (color 0 0 0 0)
+  )
+  (junction (at 78.74 60.96) (diameter 0) (color 0 0 0 0)
   )
   (junction (at 181.61 125.73) (diameter 0) (color 0 0 0 0)
@@
     (stroke (width 0) (type default))
   )
-  (wire (pts (xy 104.14 81.28) (xy 111.76 81.28))
-    (stroke (width 0) (type default))
-  )
   (wire (pts (xy 50.8 80.01) (xy 50.8 88.9))
     (stroke (width 0) (type default))
@@
     (stroke (width 0) (type default))
   )
+  (wire (pts (xy 93.98 90.17) (xy 93.98 81.28))
+    (stroke (width 0) (type default))
+  )
   (wire (pts (xy 219.71 143.51) (xy 226.06 143.51))
     (stroke (width 0) (type default))
@@
     (stroke (width 0) (type default))
   )
-  (wire (pts (xy 50.8 60.96) (xy 93.98 60.96))
+  (wire (pts (xy 111.76 90.17) (xy 93.98 90.17))
+    (stroke (width 0) (type default))
+  )
+  (wire (pts (xy 50.8 60.96) (xy 78.74 60.96))
     (stroke (width 0) (type default))
   )
@@
     (stroke (width 0) (type default))
   )
-  (wire (pts (xy 50.8 55.88) (xy 50.8 60.96))
-    (stroke (width 0) (type default))
-  )
   (wire (pts (xy 50.8 68.58) (xy 50.8 80.01))
     (stroke (width 0) (type default))
@@
     (stroke (width 0) (type default))
   )
+  (wire (pts (xy 78.74 60.96) (xy 93.98 60.96))
+    (stroke (width 0) (type default))
+  )
   (wire (pts (xy 226.06 138.43) (xy 226.06 125.73))
     (stroke (width 0) (type default))
@@
     (stroke (width 0) (type default))
   )
-  (wire (pts (xy 111.76 35.56) (xy 111.76 81.28))
+  (wire (pts (xy 111.76 35.56) (xy 111.76 90.17))
     (stroke (width 0) (type default))
   )
@@
     (stroke (width 0) (type default))
   )
-  (wire (pts (xy 68.58 55.88) (xy 50.8 55.88))
-    (stroke (width 0) (type default))
-  )
   (wire (pts (xy 38.1 60.96) (xy 40.64 60.96))
     (stroke (width 0) (type default))
@@
   )
   (wire (pts (xy 219.71 138.43) (xy 226.06 138.43))
+    (stroke (width 0) (type default))
+  )
+  (wire (pts (xy 78.74 55.88) (xy 78.74 60.96))
     (stroke (width 0) (type default))
   )
@@
   (text "+12V to transceiver" (at 252.73 152.4 90)
     (effects (font (size 1.27 1.27)) (justify left bottom))
+  )
+  (netclass_flag "" (length 2.54) (shape round) (at 227.33 140.97 0) (fields_autoplaced)
+    (effects (font (size 1.27 1.27)) (justify left bottom))
+    (property "Netclass" "12V" (at 228.0285 138.43 0)
+      (effects (font (size 1.27 1.27) italic) (justify left))
+    )
   )
   (netclass_flag "" (length 2.54) (shape round) (at 46.99 171.45 270) (fields_autoplaced)
@@
     )
   )
+  (netclass_flag "" (length 2.54) (shape round) (at 236.22 148.59 0) (fields_autoplaced)
+    (effects (font (size 1.27 1.27)) (justify left bottom))
+  )
+  (symbol (lib_id "power:GND") (at 104.14 81.28 0) (unit 1)
+    (in_bom yes) (on_board yes) (dnp no) (fields_autoplaced)
+    (property "Reference" "#PWR022" (at 104.14 87.63 0)
+      (effects (font (size 1.27 1.27)) hide)
+    )
+    (property "Value" "GND" (at 104.14 86.36 0)
+      (effects (font (size 1.27 1.27)))
+    )
+    (property "Footprint" "" (at 104.14 81.28 0)
+      (effects (font (size 1.27 1.27)) hide)
+    )
+    (property "Datasheet" "" (at 104.14 81.28 0)
+      (effects (font (size 1.27 1.27)) hide)
+    )
+    (pin "1")
+    (instances
+      (project "SWR Protector"
+        (path "/46027dd5-036f-43c6-98e1-c4cfe473ecd7"
+          (reference "#PWR022") (unit 1)
+        )
+      )
+    )
+  )
   (symbol (lib_id "power:GND") (at 46.99 184.15 0) (unit 1)
     (in_bom yes) (on_board yes) (dnp no) (fields_autoplaced)
@@
     )
   )
-  (symbol (lib_id "Device:Transformer_1P_1S") (at 99.06 71.12 270) (unit 1)
-    (in_bom yes) (on_board yes) (dnp no)
-    (property "Reference" "T2" (at 83.82 69.85 90)
-      (effects (font (size 1.27 1.27)) (justify left))
-    )
-    (property "Value" "12:1 ???" (at 83.82 72.39 90)
-      (effects (font (size 1.27 1.27) (color 255 0 0 1)) (justify left))
-    )
-    (property "Footprint" "Transformer_THT:Transformer_Toroid_Horizontal_D9.0mm_Amidon-T30" (at 99.06 71.12 0)
+  (symbol (lib_id "Device:Transformer_1P_1S") (at 99.06 71.12 90) (unit 1)
+    (in_bom yes) (on_board yes) (dnp no)
+    (property "Reference" "T2" (at 114.3 72.39 90)
+      (effects (font (size 1.27 1.27)) (justify left))
+    )
+    (property "Value" "1:12" (at 114.3 69.85 90)
+      (effects (font (size 1.27 1.27)) (justify left))
+    )
+    (property "Footprint" "FT37-43:FT37-43-TRANSFORMER" (at 99.06 71.12 0)
       (effects (font (size 1.27 1.27)) hide)
     )
@@
     )
   )
-  (symbol (lib_id "power:GND") (at 78.74 55.88 0) (unit 1)
-    (in_bom yes) (on_board yes) (dnp no)
-    (property "Reference" "#PWR021" (at 78.74 62.23 0)
-      (effects (font (size 1.27 1.27)) hide)
-    )
-    (property "Value" "GND" (at 81.28 58.42 0)
-      (effects (font (size 1.27 1.27)))
-    )
-    (property "Footprint" "" (at 78.74 55.88 0)
-      (effects (font (size 1.27 1.27)) hide)
-    )
-    (property "Datasheet" "" (at 78.74 55.88 0)
-      (effects (font (size 1.27 1.27)) hide)
-    )
-    (pin "1")
-    (instances
-      (project "SWR Protector"
-        (path "/46027dd5-036f-43c6-98e1-c4cfe473ecd7"
-          (reference "#PWR021") (unit 1)
-        )
-      )
-    )
-  )
   (symbol (lib_id "Device:R_Potentiometer") (at 121.92 146.05 0) (unit 1)
     (in_bom yes) (on_board yes) (dnp no) (fields_autoplaced)
@@
     )
   )
-  (symbol (lib_id "Device:Transformer_1P_1S") (at 73.66 45.72 270) (unit 1)
-    (in_bom yes) (on_board yes) (dnp no) (fields_autoplaced)
-    (property "Reference" "T1" (at 80.01 45.0977 90)
-      (effects (font (size 1.27 1.27)) (justify left))
-    )
-    (property "Value" "1:12" (at 80.01 47.6377 90)
-      (effects (font (size 1.27 1.27)) (justify left))
-    )
-    (property "Footprint" "Transformer_THT:Transformer_Toroid_Horizontal_D9.0mm_Amidon-T30" (at 73.66 45.72 0)
+  (symbol (lib_id "Device:Transformer_1P_1S") (at 73.66 45.72 90) (unit 1)
+    (in_bom yes) (on_board yes) (dnp no)
+    (property "Reference" "T1" (at 67.31 46.3423 90)
+      (effects (font (size 1.27 1.27)) (justify left))
+    )
+    (property "Value" "1:12" (at 67.31 43.8023 90)
+      (effects (font (size 1.27 1.27)) (justify left))
+    )
+    (property "Footprint" "FT37-43:FT37-43-TRANSFORMER" (at 73.66 45.72 0)
       (effects (font (size 1.27 1.27)) hide)
     )
@@
         (path "/46027dd5-036f-43c6-98e1-c4cfe473ecd7"
           (reference "R3") (unit 1)
+        )
+      )
+    )
+  )
+  (symbol (lib_id "power:GND") (at 68.58 55.88 270) (unit 1)
+    (in_bom yes) (on_board yes) (dnp no) (fields_autoplaced)
+    (property "Reference" "#PWR021" (at 62.23 55.88 0)
+      (effects (font (size 1.27 1.27)) hide)
+    )
+    (property "Value" "GND" (at 64.77 56.515 90)
+      (effects (font (size 1.27 1.27)) (justify right))
+    )
+    (property "Footprint" "" (at 68.58 55.88 0)
+      (effects (font (size 1.27 1.27)) hide)
+    )
+    (property "Datasheet" "" (at 68.58 55.88 0)
+      (effects (font (size 1.27 1.27)) hide)
+    )
+    (pin "1")
+    (instances
+      (project "SWR Protector"
+        (path "/46027dd5-036f-43c6-98e1-c4cfe473ecd7"
+          (reference "#PWR021") (unit 1)
         )
       )
@@
         )
       )
-    )
-  )
-  (symbol (lib_id "power:GND") (at 93.98 81.28 0) (unit 1)
-    (in_bom yes) (on_board yes) (dnp no) (fields_autoplaced)
-    (property "Reference" "#PWR022" (at 93.98 87.63 0)
-      (effects (font (size 1.27 1.27)) hide)
-    )
-    (property "Value" "GND" (at 93.98 86.36 0)
-      (effects (font (size 1.27 1.27)))
-    )
-    (property "Footprint" "" (at 93.98 81.28 0)
-      (effects (font (size 1.27 1.27)) hide)
-    )
-    (property "Datasheet" "" (at 93.98 81.28 0)
-      (effects (font (size 1.27 1.27)) hide)
-    )
-    (pin "1")
-    (instances
-      (project "SWR Protector"
-        (path "/46027dd5-036f-43c6-98e1-c4cfe473ecd7"
-          (reference "#PWR022") (unit 1)
-        )
-      )
